File: electrical/ipod_a2dp/raspberry_aux_board_connectors.brd (EAGLE design)
At the start: 30.1 x 71.1 mm, 13 parts

Commit message: update codez.
Connections:
- net IP_RX_P: now also SV2.8; no longer SV2.7
- net IP_TX_GR: now also SV2.7; no longer SV2.8
Routing:
- net IP_RX_P: track 2.68 -> 0.00 mm
- net IP_TX_GR: track 2.68 -> 4.97 mm
Changed lines of the file:
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@@
 </signal>
 <signal name="IP_TX_GR">
-<contactref element="SV2" pad="8"/>
 <contactref element="IP_5" pad="1"/>
 <wire x1="53.4924" y1="7.7724" x2="55.7784" y2="7.7724" width="0.6096" layer="1"/>
-<wire x1="55.7784" y1="7.7724" x2="55.88" y2="7.62" width="0.6096" layer="1"/>
 <wire x1="53.4924" y1="7.7724" x2="53.34" y2="7.62" width="0.6096" layer="1"/>
-</signal>
-<signal name="IP_RX_P">
 <contactref element="SV2" pad="7"/>
-<contactref element="IP_6" pad="1"/>
 <wire x1="60.8076" y1="7.7724" x2="58.5216" y2="7.7724" width="0.6096" layer="1"/>
 <wire x1="58.5216" y1="7.7724" x2="58.42" y2="7.62" width="0.6096" layer="1"/>
-<wire x1="60.8076" y1="7.7724" x2="60.96" y2="7.62" width="0.6096" layer="1"/>
+<wire x1="55.7784" y1="7.7724" x2="58.42" y2="7.62" width="0" layer="19" extent="1-1"/>
 </signal>
 <signal name="CONN_RECOG_Y">
@@
 <contactref element="IP_16" pad="1"/>
 </signal>
+<signal name="IP_RX_P">
+<contactref element="SV2" pad="8"/>
+<contactref element="IP_6" pad="1"/>
+<wire x1="55.88" y1="7.62" x2="60.96" y2="7.62" width="0" layer="19" extent="1-1"/>
+</signal>
 </signals>
