File: electrical/ipod_a2dp/raspberry_aux_board_connectors.sch (EAGLE design)
At the start: 13 parts

Commit message: update codez.
Connections:
- net IP_RX_P: now also SV2.8; no longer SV2.7
- net IP_TX_GR: now also SV2.7; no longer SV2.8
