File: electrical/ipod_a2dp/raspberry_aux_board_recover.brd (EAGLE design)
At the start: 30.1 x 71.1 mm, 31 parts, among them IC1 74LS244DW, IC2 788TV, X1 057-010-0

Commit message: update codez.
Parts:
- C7: value 220n -> 100n
- R10, R9: value 220 -> 100
- R5, R6: value 5K6 -> 10K
Connections:
- net IP_RX: now also R10.1, X1.8; no longer R9.1, X1.7
- net IP_TX: now also R9.1, X1.7; no longer R10.1, X1.8
Routing:
- net IP_TX: track 35.1 -> 54.0 mm
- net IP_RX: track 54.0 -> 35.1 mm
Changed lines of the file:
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@@
 <attribute name="VALUE" x="32.385" y="35.2806" size="1.27" layer="27" ratio="10" rot="R270"/>
 </element>
-<element name="R10" library="rcl" library_urn="urn:adsk.eagle:library:334" package="0207/10" package3d_urn="urn:adsk.eagle:package:23491/2" value="220" x="35.56" y="33.02" smashed="yes" rot="R90">
+<element name="R10" library="rcl" library_urn="urn:adsk.eagle:library:334" package="0207/10" package3d_urn="urn:adsk.eagle:package:23491/2" value="100" x="35.56" y="33.02" smashed="yes" rot="R90">
 <attribute name="NAME" x="36.195" y="31.496" size="1.27" layer="25" ratio="10" rot="R90"/>
 <attribute name="SPICEPREFIX" value="R" x="99.06" y="77.47" size="1.778" layer="27" rot="R90" display="off"/>
@@
 <attribute name="VALUE" x="37.465" y="36.5506" size="1.27" layer="27" ratio="10" rot="R270"/>
 </element>
-<element name="R5" library="rcl" library_urn="urn:adsk.eagle:library:334" package="0204/5" package3d_urn="urn:adsk.eagle:package:23488/1" value="5K6" x="22.86" y="17.78" smashed="yes">
+<element name="R5" library="rcl" library_urn="urn:adsk.eagle:library:334" package="0204/5" package3d_urn="urn:adsk.eagle:package:23488/1" value="10K" x="22.86" y="17.78" smashed="yes">
 <attribute name="NAME" x="21.463" y="17.145" size="1.27" layer="25" ratio="10"/>
 <attribute name="SPICEPREFIX" value="R" x="80.01" y="-40.64" size="1.778" layer="27" display="off"/>
 <attribute name="VALUE" x="20.5994" y="17.145" size="1.27" layer="27" ratio="10"/>
 </element>
-<element name="R6" library="rcl" library_urn="urn:adsk.eagle:library:334" package="0204/5" package3d_urn="urn:adsk.eagle:package:23488/1" value="5K6" x="22.86" y="20.32" smashed="yes">
+<element name="R6" library="rcl" library_urn="urn:adsk.eagle:library:334" package="0204/5" package3d_urn="urn:adsk.eagle:package:23488/1" value="10K" x="22.86" y="20.32" smashed="yes">
 <attribute name="NAME" x="21.717" y="19.685" size="1.27" layer="25" ratio="10"/>
 <attribute name="SPICEPREFIX" value="R" x="92.71" y="-38.1" size="1.778" layer="27" display="off"/>
 <attribute name="VALUE" x="20.5994" y="19.685" size="1.27" layer="27" ratio="10"/>
 </element>
-<element name="R9" library="rcl" library_urn="urn:adsk.eagle:library:334" package="0204/7" package3d_urn="urn:adsk.eagle:package:23498/2" value="220" x="35.56" y="46.99" smashed="yes" rot="R90">
+<element name="R9" library="rcl" library_urn="urn:adsk.eagle:library:334" package="0204/7" package3d_urn="urn:adsk.eagle:package:23498/2" value="100" x="35.56" y="46.99" smashed="yes" rot="R90">
 <attribute name="NAME" x="36.195" y="45.847" size="1.27" layer="25" ratio="10" rot="R90"/>
 <attribute name="SPICEPREFIX" value="R" x="99.06" y="78.74" size="1.778" layer="27" rot="R90" display="off"/>
@@
 <attribute name="VALUE" x="25.4" y="58.42" size="1.27" layer="27" ratio="10"/>
 </element>
-<element name="C7" library="rcl" library_urn="urn:adsk.eagle:library:334" package="C050-050X075" package3d_urn="urn:adsk.eagle:package:23665/1" value="220n" x="24.13" y="55.88" smashed="yes" rot="R180">
+<element name="C7" library="rcl" library_urn="urn:adsk.eagle:library:334" package="C050-050X075" package3d_urn="urn:adsk.eagle:package:23665/1" value="100n" x="24.13" y="55.88" smashed="yes" rot="R180">
 <attribute name="NAME" x="25.273" y="54.864" size="1.27" layer="25" ratio="10" rot="R180"/>
 <attribute name="SPICEPREFIX" value="C" x="24.13" y="55.88" size="1.778" layer="27" rot="R180" display="off"/>
@@
 <wire x1="29.21" y1="13.97" x2="35.56" y2="7.62" width="0.6096" layer="1"/>
 </signal>
-<signal name="IP_RX">
+<signal name="IP_TX">
 <contactref element="R9" pad="1"/>
 <contactref element="X1" pad="7"/>
@@
 <via x="18.415" y="34.925" extent="1-16" drill="0.7"/>
 </signal>
-<signal name="IP_TX">
+<signal name="IP_RX">
 <contactref element="R10" pad="1"/>
 <contactref element="X1" pad="8"/>
